File: schematic/Cronus.kicad_pcb (KiCad board)
At the start: 2 copper layers, 70 x 50 mm, 16 parts, among them J1 5V_In, J2 DCL, J3 DCS, J4 DD0, J5 LS1, J6 LS2, J7 GND, U1 ESP32, U2 DS3231

Commit message: Remake schematic with KiCad #3
Parts:
- removed REF** (x4): MountingHole_2.2mm_M2, MountingHole:MountingHole_2.2mm_M2
- added H1: MountingHole, MountingHole:MountingHole_2.2mm_M2, F.Cu at (108.5, 64.8)
- added H2: MountingHole, MountingHole:MountingHole_2.2mm_M2, F.Cu at (174.5, 64.8)
- added H3: MountingHole, MountingHole:MountingHole_2.2mm_M2, F.Cu at (108.5, 110.8)
- added H4: MountingHole, MountingHole:MountingHole_2.2mm_M2, F.Cu at (174.5, 110.8)
- J1: value 5V_In -> GND; footprint Connector_PinHeader_1.00mm:PinHeader_1x01_P1.00mm_Vertical -> Connector_Pin:Pin_D0.9mm_L10.0mm_W2.4mm_FlatFork
- J2: value DCL -> 5V; footprint Connector_PinHeader_1.00mm:PinHeader_1x01_P1.00mm_Vertical -> Connector_Pin:Pin_D0.9mm_L10.0mm_W2.4mm_FlatFork
- J3: value DCS -> DCL; footprint Connector_PinHeader_1.00mm:PinHeader_1x01_P1.00mm_Vertical -> Connector_Pin:Pin_D0.9mm_L10.0mm_W2.4mm_FlatFork
- J4: value DD0 -> DCS; footprint Connector_PinHeader_1.00mm:PinHeader_1x01_P1.00mm_Vertical -> Connector_Pin:Pin_D0.9mm_L10.0mm_W2.4mm_FlatFork
- J5: value LS1 -> DD0; footprint Connector_PinHeader_1.00mm:PinHeader_1x01_P1.00mm_Vertical -> Connector_Pin:Pin_D0.9mm_L10.0mm_W2.4mm_FlatFork
- J6: value LS2 -> LS1; footprint Connector_PinHeader_1.00mm:PinHeader_1x01_P1.00mm_Vertical -> Connector_Pin:Pin_D0.9mm_L10.0mm_W2.4mm_FlatFork
- J7: value GND -> LS2; footprint Connector_PinHeader_1.00mm:PinHeader_1x01_P1.00mm_Vertical -> Connector_Pin:Pin_D0.9mm_L10.0mm_W2.4mm_FlatFork
- U1: value ESP32 -> ESP32-S3
- moved J5 63.9 mm to (110.6, 80.7)
- moved J7 63.3 mm to (172.7, 101.0)
- moved J2 8.18 mm to (110.6, 73.1), turned to 0 degrees
- moved J4 7.08 mm to (110.6, 83.3), turned to 0 degrees
- moved J3 7.08 mm to (110.6, 85.8), turned to 0 degrees
- moved J6 3.62 mm to (172.7, 98.5)
- moved R1 1.41 mm to (156.8, 101.0)
- moved R2 1.41 mm to (139.0, 98.5)
- moved R3 1.41 mm to (163.0, 98.4)
- moved U1 1.41 mm to (141.1, 76.8)
- moved U2 1.41 mm to (149.9, 102.3)
- moved J1 0.66 mm to (110.6, 70.6), turned to 0 degrees
Connections:
- J1 pad 1: +5V -> GND
- J2 pad 1: Net-(J2-Pin_1) -> +5V
- J7 pad 1: GND -> Net-(J7-Pin_1)
- R1 pad 1: Net-(J6-Pin_1) -> Net-(J7-Pin_1)
- R2 pad 1: Net-(J6-Pin_1) -> Net-(J7-Pin_1)
- R3 pad 1: Net-(J5-Pin_1) -> Net-(J6-Pin_1)
- U1 pad 1: Net-(J6-Pin_1) -> Net-(J7-Pin_1)
- U1 pad 10: Net-(J3-Pin_1) -> Net-(J4-Pin_1)
- U1 pad 11: Net-(J4-Pin_1) -> Net-(J5-Pin_1)
- U1 pad 41: Net-(J5-Pin_1) -> Net-(J6-Pin_1)
- U1 pad 9: Net-(J2-Pin_1) -> Net-(J3-Pin_1)
- U2 pad 2: Net-(J6-Pin_1) -> Net-(J7-Pin_1)
Routing:
- net Net-(J7-Pin_1): track 0.00 -> 63.6 mm
- net Net-(J2-Pin_1): track 49.1 -> 0.00 mm
- net Net-(J6-Pin_1): track 62.9 -> 31.4 mm
- net Net-(J5-Pin_1): track 31.0 -> 41.5 mm
- net GND: track 40.8 -> 47.0 mm
- net Net-(U1-GPIO38): track 23.1 -> 26.8 mm
- net Net-(J4-Pin_1): track 42.1 -> 44.8 mm
- net Net-(J3-Pin_1): track 45.6 -> 48.2 mm
- net +5V: track 10.8 -> 13.2 mm
- net unconnected-(U1-GPIO15-Pad8): track 0.00 -> 0.56 mm
Other:
- board text added: "Cronus"
- board text added: "https://cronus.d5y.xyz"
- board text added: "rev 0.1"

Commit message: Update schematic
Parts:
- J2: value 5V -> 5V_In
- R3: value 1K -> 3K
Changed lines of the file:
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@@
 			)
 		)
-		(property "Value" "5V"
+		(property "Value" "5V_In"
 			(at 0 2.54 0)
 			(layer "F.SilkS")
@@
 		(property "Value" "10K"
 			(at 0 2 0)
-			(layer "B.Fab")
+			(layer "B.SilkS")
 			(effects
 				(font
@@
 		(property "Value" "10K"
 			(at 0 -1.82 0)
-			(layer "B.Fab")
+			(layer "B.SilkS")
 			(effects
 				(font
@@
 		(tags "resistor handsolder")
 		(property "Reference" "R3"
-			(at 0 1.82 0)
+			(at 0.016 -1.959 0)
 			(layer "B.SilkS")
 			(effects
@@
 			)
 		)
-		(property "Value" "1K"
-			(at 0 -1.82 0)
-			(layer "B.Fab")
-			(effects
-				(font
+		(property "Value" "3K"
+			(at -0.111 2.105 0)
+			(layer "B.SilkS")
+			(effects
+				(font

Commit message: Update schematic
Changed lines of the file:
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@@
 	(net 13 "unconnected-(U1-GPIO3-Pad13)")
 	(net 14 "unconnected-(U1-GPIO2-Pad40)")
-	(net 15 "unconnected-(U1-GPIO15-Pad30)")
+	(net 15 "unconnected-(U1-GPIO45-Pad30)")
 	(net 16 "unconnected-(U1-RX-Pad42)")
 	(net 17 "unconnected-(U1-GPIO41-Pad38)")
@@
 			(layer "F.SilkS")
 		)
+		(fp_text user "${REFERENCE}"
+			(at 0 2.5 -90)
+			(unlocked yes)
+			(layer "F.Fab")
+			(effects
+				(font
+					(size 1 1)
+					(thickness 0.15)
+				)
+			)
+		)
 		(pad "1" thru_hole rect
 			(at -12.7 -27.94 270)
@@
 			(pintype "power_out")
 		)
-		(pad "1" thru_hole rect
+		(pad "2" thru_hole rect
 			(at -12.7 -25.4 270)
 			(size 1.6 1.6)
@@
 			(pintype "passive")
 		)
-		(pad "22" thru_hole rect
-			(at 12.7 -27.94 270)
+		(pad "23" thru_hole rect
+			(at 12.7 25.4 270)
 			(size 1.6 1.6)
 			(drill 1)
@@
 			(pintype "passive")
 		)
-		(pad "22" thru_hole rect
+		(pad "24" thru_hole rect
 			(at 12.7 22.86 270)
 			(size 1.6 1.6)
@@
 			(pintype "passive")
 		)
-		(pad "22" thru_hole rect
-			(at 12.7 25.4 270)
-			(size 1.6 1.6)
-			(drill 1)
-			(layers "*.Cu" "*.Mask")
-			(remove_unused_layers no)
-			(net 21 "GND")
-			(pinfunction "GND")
-			(pintype "passive")
-		)
 		(pad "25" thru_hole rect
 			(at 12.7 20.32 270)
@@
 			(layers "*.Cu" "*.Mask")
 			(remove_unused_layers no)
-			(net 15 "unconnected-(U1-GPIO15-Pad30)")
-			(pinfunction "GPIO15")
+			(net 15 "unconnected-(U1-GPIO45-Pad30)")
+			(pinfunction "GPIO45")
 			(pintype "bidirectional+no_connect")
 		)
@@
 			(pintype "bidirectional+no_connect")
 		)
+		(pad "44" thru_hole rect
+			(at 12.7 -27.94 270)
+			(size 1.6 1.6)
+			(drill 1)
+			(layers "*.Cu" "*.Mask")
+			(remove_unused_layers no)
+			(net 21 "GND")
+			(pinfunction "GND")
+			(pintype "passive")
+		)
 	)
 	(footprint "Connector_Pin:Pin_D0.9mm_L10.0mm_W2.4mm_FlatFork"
@@
 			(layer "F.SilkS")
 		)
-		(pad "1" thru_hole rect
-			(at 3.81 19.05 90)
-			(size 1.6 1.6)
-			(drill 1)
-			(layers "*.Cu" "*.Mask")
-			(remove_unused_layers no)
-			(net 21 "GND")
-			(pinfunction "GND")
-			(pintype "passive")
+		(fp_text user "${REFERENCE}"
+			(at 0 2.5 90)
+			(unlocked yes)
+			(layer "F.Fab")
+			(effects
+				(font
+					(size 1 1)
+					(thickness 0.15)
+				)
+			)
 		)
 		(pad "1" thru_hole rect
@@
 		)
 		(pad "2" thru_hole rect
-			(at 1.27 19.05 90)
-			(size 1.6 1.6)
-			(drill 1)
-			(layers "*.Cu" "*.Mask")
-			(remove_unused_layers no)
-			(net 37 "Net-(J7-Pin_1)")
-			(pinfunction "VCC")
-			(pintype "power_in")
-		)
-		(pad "2" thru_hole rect
 			(at 3.81 -16.51 90)
 			(size 1.6 1.6)
@@
 			(pintype "bidirectional+no_connect")
 		)
+		(pad "9" thru_hole rect
+			(at 1.27 19.05 90)
+			(size 1.6 1.6)
+			(drill 1)
+			(layers "*.Cu" "*.Mask")
+			(remove_unused_layers no)
+			(net 37 "Net-(J7-Pin_1)")
+			(pinfunction "VCC")
+			(pintype "power_in")
+		)
+		(pad "10" thru_hole rect
+			(at 3.81 19.05 90)
+			(size 1.6 1.6)
+			(drill 1)
+			(layers "*.Cu" "*.Mask")
+			(remove_unused_layers no)
+			(net 21 "GND")
+			(pinfunction "GND")
+			(pintype "passive")
+		)
 	)
 	(footprint "MountingHole:MountingHole_2.2mm_M2"
@@
 	)
 	(gr_text "rev 0.1"
-		(at 114.644 110.956 0)
+		(at 118.835 106.892 0)
 		(layer "F.SilkS")
 		(effects

Commit message: Update schematic
Parts:
- U2: footprint Cronus:DS3232-Dev-Board -> Cronus:DS3231-Dev-Board
Changed lines of the file:
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@@
 		(at 141.1 76.8 -90)
 		(property "Reference" "U1"
-			(at 0 0 0)
+			(at 0.374 2.7 90)
 			(unlocked yes)
 			(layer "F.SilkS")
@@
 		)
 		(property "Value" "ESP32-S3"
-			(at 2.152 0 0)
+			(at 0.374 0.548 90)
 			(unlocked yes)
 			(layer "F.SilkS")
@@
 		)
 		(fp_text user "${REFERENCE}"
-			(at 0 2.5 -90)
+			(at 0.414 -1.23 90)
 			(unlocked yes)
 			(layer "F.Fab")
@@
 		)
 	)
-	(footprint "Cronus:DS3232-Dev-Board"
+	(footprint "Cronus:DS3231-Dev-Board"
 		(layer "F.Cu")
 		(at 149.95 102.27 90)
 		(property "Reference" "U2"
-			(at 0.704 0.304 0)
+			(at 0 -0.5 90)
 			(unlocked yes)
 			(layer "F.SilkS")
@@
 		)
 		(property "Value" "DS3231"
-			(at -1.574 0.304 0)
-			(unlocked yes)
-			(layer "F.SilkS")
-			(effects
-				(font
-					(size 1 1)
-					(thickness 0.15)
-				)
-			)
-		)
-		(property "Footprint" "Cronus:DS3232-Dev-Board"
+			(at 0 1 90)
+			(unlocked yes)
+			(layer "F.SilkS")
+			(effects
+				(font
+					(size 1 1)
+					(thickness 0.15)
+				)
+			)
+		)
+		(property "Footprint" "Cronus:DS3231-Dev-Board"
 			(at 0 0 90)
 			(unlocked yes)

Commit message: Fix PCB
Other:
- board text added: "rev 0.2"
- board text removed: "rev 0.1"

Commit message: Upd PCB
Parts:
- removed H2: MountingHole, MountingHole:MountingHole_2.2mm_M2
- H1, H3, H4: footprint MountingHole:MountingHole_2.2mm_M2 -> MountingHole:MountingHole_2.1mm
- moved R2 19.0 mm to (152.1, 84.8), turned to -90 degrees
- moved R1 16.3 mm to (154.7, 84.8), turned to -90 degrees
- moved R3 14.3 mm to (167.4, 84.8), turned to 90 degrees
- moved J3 13.7 mm to (116.3, 73.4)
- moved J5 12.3 mm to (116.3, 69.8)
- moved J4 11.8 mm to (112.8, 71.6)
- moved J2 10.3 mm to (116.3, 64.5)
- moved J1 6.44 mm to (112.8, 64.5)
- moved U1 5.98 mm to (147.1, 77.2)
- moved U2 2.20 mm to (152.1, 102.1)
- moved J6 1.63 mm to (174.2, 98.0)
- moved J7 1.59 mm to (174.2, 100.8)
Routing:
- net Net-(J7-Pin_1): track 63.6 -> 156.3 mm, vias 0 -> 1
- net GND: track 47.0 -> 0.00 mm
- net Net-(J6-Pin_1): track 31.4 -> 17.3 mm
- net Net-(J3-Pin_1): track 48.2 -> 42.9 mm
- net Net-(J5-Pin_1): track 41.5 -> 36.2 mm
- net Net-(U1-GPIO39): track 33.8 -> 30.8 mm
- net +5V: track 13.2 -> 11.1 mm
- net Net-(J4-Pin_1): track 44.8 -> 43.1 mm
- net unconnected-(U1-GPIO15-Pad8): track 0.56 -> 0.00 mm
- added copper zone on B.Cu, net GND
Other:
- board text added: "3V3"

Commit message: Update PCB
Parts:
- removed J1: GND, Connector_Pin:Pin_D0.9mm_L10.0mm_W2.4mm_FlatFork
- removed J2: 5V_In, Connector_Pin:Pin_D0.9mm_L10.0mm_W2.4mm_FlatFork
- removed J5: DD0, Connector_Pin:Pin_D0.9mm_L10.0mm_W2.4mm_FlatFork
- removed J6: LS1, Connector_Pin:Pin_D0.9mm_L10.0mm_W2.4mm_FlatFork
- removed J7: LS2, Connector_Pin:Pin_D0.9mm_L10.0mm_W2.4mm_FlatFork
- added J8: Conn_01x03_Pin, Connector_PinHeader_2.54mm:PinHeader_1x03_P2.54mm_Vertical, F.Cu at (113.1, 84.9)
- H1, H3, H4: footprint MountingHole:MountingHole_2.1mm -> MountingHole:MountingHole_2.2mm_M2_DIN965_Pad
- J3: value DCL -> Conn_01x02_Pin; footprint Connector_Pin:Pin_D0.9mm_L10.0mm_W2.4mm_FlatFork -> Connector_PinHeader_2.54mm:PinHeader_1x02_P2.54mm_Vertical
- J4: value DCS -> Conn_01x02_Pin; footprint Connector_Pin:Pin_D0.9mm_L10.0mm_W2.4mm_FlatFork -> Connector_PinHeader_2.54mm:PinHeader_1x02_P2.54mm_Vertical
- moved J3 64.0 mm to (174.2, 100.8), turned to 180 degrees
- moved J4 2.72 mm to (113.0, 68.9)
- moved U2 0.17 mm to (152.1, 101.9)
Connections:
- J3 pad 1: Net-(J3-Pin_1) -> Net-(J3-LS1)
- J4 pad 1: Net-(J4-Pin_1) -> +5V
- R1 pad 1: Net-(J7-Pin_1) -> Net-(J3-LS1)
- R2 pad 1: Net-(J7-Pin_1) -> Net-(J3-LS1)
- R3 pad 1: Net-(J6-Pin_1) -> Net-(J3-LS2)
- U1 pad 1: Net-(J7-Pin_1) -> Net-(J3-LS1)
- U1 pad 10: Net-(J4-Pin_1) -> Net-(J8-CS)
- U1 pad 2: Net-(J7-Pin_1) -> Net-(J3-LS1)
- U1 pad 41: Net-(J6-Pin_1) -> Net-(J3-LS2)
- U1 pad 9: Net-(J3-Pin_1) -> Net-(J8-CL)
- U2 pad 2: Net-(J7-Pin_1) -> Net-(J3-LS1)
- U2 pad 9: Net-(J7-Pin_1) -> Net-(J3-LS1)
Routing:
- net Net-(J7-Pin_1): track 156.3 -> 0.00 mm, vias 1 -> 0
- net Net-(J3-LS1): track 0.00 -> 141.7 mm, vias 0 -> 1
- net Net-(J8-CL): track 0.00 -> 50.8 mm
- net Net-(J8-CS): track 0.00 -> 47.1 mm
- net Net-(J4-Pin_1): track 43.1 -> 0.00 mm
- net Net-(J3-Pin_1): track 42.9 -> 0.00 mm
- net Net-(J6-Pin_1): track 17.3 -> 0.00 mm
- net Net-(J3-LS2): track 0.00 -> 14.8 mm
- net Net-(J8-D0): track 36.2 -> 43.6 mm
- net +5V: track 11.1 -> 14.5 mm
Other:
- board text added: "+5V"
- board text added: "CL"
- board text added: "CS"
- board text added: "D0"
- board text added: "GND"
- board text added: "LS1"
- board text added: "LS2"
